Commit message: tried stuff out in unity

File: Unity/Quest3XRSApp/Assets/URDF/xArm7URDF-main/xarm7.urdf (robot description, URDF)
Before this commit: robot UF_ROBOT, 10 links, 9 joints
Links:
- link link7: geometry collision mesh filename=link7.stl; visual mesh filename=link7.stl

Commit message: added the xarm robot to unity, connected ros and unity, fixed the gravity ddragging the robot down issue

File: Unity/Quest3XRSApp/Assets/URDF/xArm7URDF-main/xarm7.urdf (robot description, URDF)
Before this commit: robot UF_ROBOT, 10 links, 9 joints
Links:
- added link left_finger; collision mesh filename=left_finger.stl; visual mesh filename=left_finger.stl
- added link left_inner_knuckle; collision mesh filename=left_inner_knuckle.stl; visual mesh filename=left_inner_knuckle.stl
- added link left_outer_knuckle; collision mesh filename=left_outer_knuckle.stl; visual mesh filename=left_outer_knuckle.stl
- added link right_finger; collision mesh filename=right_finger.stl; visual mesh filename=right_finger.stl
- added link right_inner_knuckle; collision mesh filename=right_inner_knuckle.stl; visual mesh filename=right_inner_knuckle.stl
- added link right_outer_knuckle; collision mesh filename=right_outer_knuckle.stl; visual mesh filename=right_outer_knuckle.stl
- added link xarm_gripper_base_link; collision mesh filename=base_link_collision.stl; visual mesh filename=base_link.stl
Joints:
- added joint drive_joint: type revolute, parent xarm_gripper_base_link, child left_outer_knuckle, origin xyz=0 0.035 0.059098 rpy=0 0 0, axis 1 0 0, limit lower=0 upper=0.85 effort=50 velocity=2
- added joint gripper_fix: type fixed, parent link7, child xarm_gripper_base_link, origin xyz=0 0 0 rpy=0 0 0
- added joint left_finger_joint: type revolute, parent left_outer_knuckle, child left_finger, origin xyz=0 0.035465 0.042039 rpy=0 0 0, axis -1 0 0, limit lower=0 upper=0.85 effort=50 velocity=2
- added joint left_inner_knuckle_joint: type revolute, parent xarm_gripper_base_link, child left_inner_knuckle, origin xyz=0 0.02 0.074098 rpy=0 0 0, axis 1 0 0, limit lower=0 upper=0.85 effort=50 velocity=2
- added joint right_finger_joint: type revolute, parent right_outer_knuckle, child right_finger, origin xyz=0 -0.035465 0.042039 rpy=0 0 0, axis 1 0 0, limit lower=0 upper=0.85 effort=50 velocity=2
- added joint right_inner_knuckle_joint: type revolute, parent xarm_gripper_base_link, child right_inner_knuckle, origin xyz=0 -0.02 0.074098 rpy=0 0 0, axis -1 0 0, limit lower=0 upper=0.85 effort=50 velocity=2
- added joint right_outer_knuckle_joint: type revolute, parent xarm_gripper_base_link, child right_outer_knuckle, origin xyz=0 -0.035 0.059098 rpy=0 0 0, axis -1 0 0, limit lower=0 upper=0.85 effort=50 velocity=2
